File: bc29.brd (EAGLE design)
At the start: 116.8 x 86.4 mm, 107 parts, among them J1 2520-5, Q1 IRF740, U1 LP2951, U10 MC14516B, U11 CD4053B, U12 HCF4520, U13 CD4013B, U14 CD4070B, U15 TSC900BIJA, U16 CD4060B, U17 MC14073B, U18 CD4070B, U19 CD4001B, U2 CD4081, U3 CD4023, U4 CD4093B, U5 MC14516B, U6 CD4013, U7 TLC27L41, U8 CD4013B, U9 CD4001B, X1 32.768KHz

Commit message: more charge/discharge
Connections:
- net DISCHAR renamed DISCHARGE
- net N$13 renamed LCD-3
- net N$14 renamed LCD-10
- net N$15 renamed LCD-1
- net N$16 renamed LCD-8
- net N$17 renamed LCD-7
- net N$18 renamed LCD-9
- net N$19 renamed LCD-11
- net N$20 renamed LCD-13
- net N$21 renamed LCD-15
- net N$22 renamed LCD-17
- net N$23 renamed LCD-19
- net N$26 renamed LCD-18
- net N$28 renamed LCD-16
- net N$30 renamed IN-
- net N$31 renamed VDD+
- net N$33 renamed VDD-
- net N$34 renamed OUT
- net N$36 renamed IN+
- net N$41 renamed CXA
- net N$43 renamed CXB
- net N$46 renamed -2V5_BUF_R
- net N$47 renamed -2V5_BUF
- net RESET: now also U13.10, U13.4, U5.9, U6.10
Changed lines of the file:
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@@
 <wire x1="6.35" y1="71.12" x2="12.7" y2="67.31" width="0" layer="19" extent="1-1"/>
 </signal>
-<signal name="N$15">
+<signal name="LCD-1">
 <contactref element="J1" pad="1"/>
 <contactref element="U18" pad="10"/>
@@
 <signal name="RESET">
 <contactref element="U4" pad="4"/>
+<contactref element="U6" pad="10"/>
+<contactref element="U5" pad="9"/>
+<contactref element="U13" pad="4"/>
+<contactref element="U13" pad="10"/>
+<wire x1="86.995" y1="66.5734" x2="99.06" y2="66.5734" width="0" layer="19" extent="1-1"/>
+<wire x1="78.74" y1="36.0934" x2="86.995" y2="66.5734" width="0" layer="19" extent="1-1"/>
+<wire x1="77.47" y1="29.9466" x2="78.74" y2="36.0934" width="0" layer="19" extent="1-1"/>
+<wire x1="54.61" y1="57.8866" x2="78.74" y2="36.0934" width="0" layer="19" extent="1-1"/>
 </signal>
 <signal name="AH_NEGATIVE">
@@
 <wire x1="6.35" y1="15.24" x2="12.7" y2="39.37" width="0" layer="19" extent="1-1"/>
 </signal>
-<signal name="N$13">
+<signal name="LCD-3">
 <contactref element="J1" pad="3"/>
 <contactref element="U2" pad="4"/>
@@
 <wire x1="82.55" y1="73.1266" x2="101.6" y2="53.34" width="0" layer="19" extent="1-1"/>
 </signal>
-<signal name="N$16">
+<signal name="LCD-8">
 <contactref element="U14" pad="4"/>
 <contactref element="J1" pad="8"/>
 <wire x1="92.71" y1="29.9466" x2="107.95" y2="48.26" width="0" layer="19" extent="1-1"/>
 </signal>
-<signal name="N$17">
+<signal name="LCD-7">
 <contactref element="U14" pad="11"/>
 <contactref element="J1" pad="7"/>
 <wire x1="92.71" y1="36.0934" x2="105.41" y2="48.26" width="0" layer="19" extent="1-1"/>
 </signal>
-<signal name="N$18">
+<signal name="LCD-9">
 <contactref element="U17" pad="10"/>
 <contactref element="J1" pad="9"/>
@@
 <wire x1="83.82" y1="23.3934" x2="105.41" y2="45.72" width="0" layer="19" extent="1-1"/>
 </signal>
-<signal name="N$14">
+<signal name="LCD-10">
 <contactref element="U14" pad="10"/>
 <contactref element="J1" pad="10"/>
@@
 <wire x1="107.95" y1="40.64" x2="78.74" y2="73.1266" width="0" layer="19" extent="1-1"/>
 </signal>
-<signal name="N$19">
+<signal name="LCD-11">
 <contactref element="J1" pad="11"/>
 <contactref element="U14" pad="3"/>
 <wire x1="91.44" y1="29.9466" x2="105.41" y2="43.18" width="0" layer="19" extent="1-1"/>
 </signal>
-<signal name="N$20">
+<signal name="LCD-13">
 <contactref element="J1" pad="13"/>
 <contactref element="U3" pad="9"/>
 <wire x1="105.41" y1="40.64" x2="100.33" y2="79.2734" width="0" layer="19" extent="1-1"/>
 </signal>
-<signal name="N$21">
+<signal name="LCD-15">
 <contactref element="J1" pad="15"/>
 <contactref element="U18" pad="3"/>
@@
 <wire x1="96.52" y1="17.2466" x2="105.41" y2="38.1" width="0" layer="19" extent="1-1"/>
 </signal>
-<signal name="N$22">
+<signal name="LCD-17">
 <contactref element="U11" pad="4"/>
 <contactref element="J1" pad="17"/>
 <wire x1="34.925" y1="37.5666" x2="105.41" y2="35.56" width="0" layer="19" extent="1-1"/>
 </signal>
-<signal name="N$23">
+<signal name="LCD-19">
 <contactref element="U14" pad="5"/>
 <contactref element="U14" pad="2"/>
@@
 <wire x1="93.345" y1="48.7934" x2="96.52" y2="51.64" width="0" layer="19" extent="1-1"/>
 </signal>
-<signal name="N$26">
+<signal name="LCD-18">
+<contactref element="U4" pad="9"/>
+<contactref element="J1" pad="18"/>
 <contactref element="U18" pad="9"/>
-<contactref element="J1" pad="18"/>
-<contactref element="U4" pad="9"/>
 <wire x1="100.33" y1="23.3934" x2="107.95" y2="35.56" width="0" layer="19" extent="1-1"/>
 <wire x1="57.15" y1="64.0334" x2="107.95" y2="35.56" width="0" layer="19" extent="1-1"/>
 </signal>
-<signal name="N$28">
+<signal name="LCD-16">
 <contactref element="J1" pad="16"/>
 <contactref element="U19" pad="3"/>
@@
 <wire x1="59.055" y1="9.6266" x2="51.435" y2="29.9466" width="0" layer="19" extent="1-1"/>
 </signal>
-<signal name="N$36">
+<signal name="IN+">
 <contactref element="R25" pad="2"/>
 <contactref element="C17" pad="1"/>
@@
 <wire x1="15.24" y1="14.29" x2="15.24" y2="22.86" width="0" layer="19" extent="1-1"/>
 </signal>
-<signal name="N$30">
+<signal name="IN-">
 <contactref element="R19" pad="2"/>
 <contactref element="U15" pad="2"/>
@@
 <wire x1="26.67" y1="13.02" x2="15.24" y2="16.19" width="0" layer="19" extent="1-1"/>
 </signal>
-<signal name="N$31">
+<signal name="VDD+">
 <contactref element="R26" pad="1"/>
 <contactref element="U15" pad="7"/>
@@
 <wire x1="52.07" y1="3.68" x2="51.12" y2="13.97" width="0" layer="19" extent="1-1"/>
 </signal>
-<signal name="N$33">
+<signal name="VDD-">
 <contactref element="U15" pad="4"/>
 <contactref element="R27" pad="2"/>
@@
 <wire x1="55.88" y1="3.68" x2="51.12" y2="10.16" width="0" layer="19" extent="1-1"/>
 </signal>
-<signal name="N$41">
+<signal name="CXA">
 <contactref element="U15" pad="1"/>
 <contactref element="C13" pad="1"/>
 <wire x1="44.45" y1="3.68" x2="39.37" y2="19.05" width="0" layer="19" extent="1-1"/>
 </signal>
-<signal name="N$43">
+<signal name="CXB">
 <contactref element="U15" pad="8"/>
 <contactref element="C14" pad="1"/>
 <wire x1="48.26" y1="3.68" x2="46.99" y2="19.05" width="0" layer="19" extent="1-1"/>
 </signal>
-<signal name="N$34">
+<signal name="OUT">
 <contactref element="U15" pad="6"/>
 <contactref element="C11" pad="2"/>
@@
 <wire x1="26.67" y1="21.59" x2="36.83" y2="24.13" width="0" layer="19" extent="1-1"/>
 </signal>
-<signal name="N$46">
+<signal name="-2V5_BUF_R">
 <contactref element="U11" pad="14"/>
 <contactref element="R13" pad="1"/>
 <wire x1="33.655" y1="43.7134" x2="37.15" y2="46.99" width="0" layer="19" extent="1-1"/>
 </signal>
-<signal name="N$47">
+<signal name="-2V5_BUF">
 <contactref element="R13" pad="2"/>
 <contactref element="U7" pad="7"/>
@@
 <wire x1="76.2" y1="42.6466" x2="81.28" y2="79.2734" width="0" layer="19" extent="1-1"/>
 </signal>
-<signal name="DISCHAR">
+<signal name="DISCHARGE">
 <contactref element="U8" pad="13"/>
 <contactref element="U11" pad="11"/>

Commit message: Digital updates
Connections:
- net LCD-15 renamed !UP_DOWN_CLK
- net N$27 renamed SHUNT+FILTER
- net N$35 renamed X0
- net N$37 renamed Y0
- removed net LCD-1: J1.1, U18.10
- removed net N$25: D5.A, U10.12
- removed net N$52: U10.15, U5.15
- new net !DOWN: J1.1, U10.10, U17.11, U18.10, U18.13, U5.10, U9.6
- new net N$13: U10.3, U14.13
- new net N$14: U10.7, U6.5, U6.6
- new net N$15: U10.9
- new net N$16: U14.6, U18.8
- new net N$17: U10.1, U6.2
- new net N$18: U3.6, U6.8, U6.9
- new net N$19: U10.5, U5.7
- new net UP_DOWN_CLK: U10.15, U3.10, U5.15, U6.11, U6.3
- net +5V: now also U3.12, U3.13
- net GND: now also D5.A, U10.12, U10.13, U10.4, U5.1, U5.12, U5.13, U5.3, U5.4
- net RESET: now also U11.9

Commit message: cleanup up/down counter
Connections:
- net LCD-18 renamed AH_NEGATIVE_LCD
- net N$50 renamed OUT-_R
- net N$58 renamed OUT+_R
- removed net N$49: R17.2, U13.6
- removed net N$51: C19.1, R1.2, R6.1
- removed net N$59: U2.2, U9.11
- removed net N$60: U19.8, U9.2
- removed net N$61: U2.12, U9.3
- removed net U13-1: R3.2, R6.2, U13.1
- removed net U8-SET: C25.1, R17.1, U4.12, U8.6, U8.8
- new net !1_024KHZ: U4.11, U8.11, U8.3
- new net !NAR_R: C19.1, R1.2, R6.1, U4.8
- new net !OUT+: U18.2, U19.1, U2.12, U9.3
- new net !OUT-: U18.1, U19.13, U2.2, U9.11
- new net AH_NEGATIVE_R: R3.2, R6.2, U13.1, U14.6, U18.8
- new net N$20: U8.2, U9.8
- new net N$21: U8.12, U9.9
- new net N$22: U19.11, U19.2
- new net N$23: U12.6, U12.9
- new net N$26: U17.6, U18.5
- new net N$27: U13.13, U17.12, U18.12, U18.6
- new net U12-14: U12.1, U12.14, U19.8, U9.12, U9.2
- net +5V: now also U10.3, U12.10, U14.13, U17.13
- net 1_024KHZ: now also U4.12, U8.6, U8.8; no longer U8.11, U8.3
- net GND: now also R17.2, U13.6, U13.8
- net LCD-16: now also U13.5, U19.12
- net N$13: now also C25.2, U9.10; no longer U10.3, U14.13
- net N$15: now also U6.12
- net N$16: now also U13.9, U18.4; no longer U14.6, U18.8
- net N$24: now also C25.1, R17.1, U12.15, U12.7; no longer C25.2, U19.10
- net UP_DOWN_CLK: now also U13.11, U9.5

Commit message: cleanup random gates
Connections:
- removed net N$18: U3.6, U6.8, U6.9
- removed net N$19: U10.5, U5.7
- removed net N$27: U13.13, U17.12, U18.12, U18.6
- new net N$25: U19.10, U19.5
- new net U13-12: U13.12, U17.1
- new net U13-13: U13.13, U14.8, U17.12, U18.12, U18.6
- new net U13-3: U13.3, U17.9
- new net U14-1: U14.1, U19.4, U19.9
- new net U17-2: U17.2, U17.3, U17.4, U2.4
- new net U3-6: U3.6, U3.8, U6.8, U6.9
- new net U4-3: U3.5, U4.3
- new net U5-7: U10.5, U4.1, U4.2, U5.7
- new net U6-5: U10.7, U3.1, U3.2, U6.5, U6.6
- new net U9-4: U17.8, U9.4
- net !DOWN: now also U3.4
- net !OUT-: now also U3.3
- net !UP_DOWN_CLK: now also U19.6
- net LCD-13: now also U2.5
- net LCD-3: now also U2.6; no longer U2.4
- net N$14: now also U17.5, U18.11; no longer U10.7, U6.5, U6.6
Changed lines of the file:
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@@
 <signal name="LCD-3">
 <contactref element="J1" pad="3"/>
-<contactref element="U2" pad="4"/>
 <contactref element="C1" pad="1"/>
+<contactref element="U2" pad="6"/>
 <wire x1="101.6" y1="53.34" x2="105.41" y2="53.34" width="0" layer="19" extent="1-1"/>
-<wire x1="82.55" y1="73.1266" x2="101.6" y2="53.34" width="0" layer="19" extent="1-1"/>
+<wire x1="85.09" y1="73.1266" x2="101.6" y2="53.34" width="0" layer="19" extent="1-1"/>
 </signal>
 <signal name="LCD-8">
@@
 <contactref element="J1" pad="13"/>
 <contactref element="U3" pad="9"/>
+<contactref element="U2" pad="5"/>
+<wire x1="83.82" y1="73.1266" x2="100.33" y2="79.2734" width="0" layer="19" extent="1-1"/>
 <wire x1="105.41" y1="40.64" x2="100.33" y2="79.2734" width="0" layer="19" extent="1-1"/>
 </signal>
@@
 <contactref element="U18" pad="3"/>
 <contactref element="U3" pad="11"/>
+<contactref element="U19" pad="6"/>
 <wire x1="105.41" y1="38.1" x2="97.79" y2="79.2734" width="0" layer="19" extent="1-1"/>
 <wire x1="96.52" y1="17.2466" x2="105.41" y2="38.1" width="0" layer="19" extent="1-1"/>
+<wire x1="85.09" y1="4.5466" x2="96.52" y2="17.2466" width="0" layer="19" extent="1-1"/>
 </signal>
 <signal name="LCD-17">
@@
 <signal name="DISCHARGE">
 <contactref element="U11" pad="11"/>
+<contactref element="U8" pad="13"/>
 <contactref element="U9" pad="13"/>
-<contactref element="U8" pad="13"/>
 <wire x1="52.07" y1="48.7934" x2="74.93" y2="48.7934" width="0" layer="19" extent="1-1"/>
 <wire x1="37.465" y1="43.7134" x2="52.07" y2="48.7934" width="0" layer="19" extent="1-1"/>
 </signal>
 <signal name="CHARGE">
-<contactref element="U9" pad="1"/>
 <contactref element="U11" pad="10"/>
 <contactref element="U8" pad="1"/>
+<contactref element="U9" pad="1"/>
 <wire x1="50.8" y1="42.6466" x2="73.66" y2="42.6466" width="0" layer="19" extent="1-1"/>
 <wire x1="38.735" y1="43.7134" x2="50.8" y2="42.6466" width="0" layer="19" extent="1-1"/>
-</signal>
-<signal name="N$14">
-<contactref element="U10" pad="7"/>
-<contactref element="U6" pad="6"/>
-<contactref element="U6" pad="5"/>
-<wire x1="99.06" y1="60.4266" x2="100.33" y2="60.4266" width="0" layer="19" extent="1-1"/>
-<wire x1="95.885" y1="42.6466" x2="99.06" y2="60.4266" width="0" layer="19" extent="1-1"/>
 </signal>
 <signal name="N$15">
@@
 <contactref element="U10" pad="1"/>
 <wire x1="88.265" y1="42.6466" x2="95.25" y2="60.4266" width="0" layer="19" extent="1-1"/>
-</signal>
-<signal name="N$18">
-<contactref element="U6" pad="8"/>
-<contactref element="U6" pad="9"/>
-<contactref element="U3" pad="6"/>
-<wire x1="100.33" y1="66.5734" x2="100.33" y2="73.1266" width="0" layer="19" extent="1-1"/>
-<wire x1="101.6" y1="66.5734" x2="100.33" y2="66.5734" width="0" layer="19" extent="1-1"/>
-</signal>
-<signal name="N$19">
-<contactref element="U10" pad="5"/>
-<contactref element="U5" pad="7"/>
-<wire x1="93.345" y1="42.6466" x2="85.725" y2="60.4266" width="0" layer="19" extent="1-1"/>
 </signal>
 <signal name="!DOWN">
@@
 <contactref element="U18" pad="10"/>
 <contactref element="U18" pad="13"/>
+<contactref element="U3" pad="4"/>
+<wire x1="85.725" y1="66.5734" x2="97.79" y2="73.1266" width="0" layer="19" extent="1-1"/>
+<wire x1="105.41" y1="55.88" x2="97.79" y2="73.1266" width="0" layer="19" extent="1-1"/>
 <wire x1="95.885" y1="48.7934" x2="105.41" y2="55.88" width="0" layer="19" extent="1-1"/>
 <wire x1="80.01" y1="42.6466" x2="95.885" y2="48.7934" width="0" layer="19" extent="1-1"/>
@@
 <wire x1="95.25" y1="23.3934" x2="82.55" y2="23.3934" width="0" layer="19" extent="1-1"/>
 <wire x1="99.06" y1="23.3934" x2="95.25" y2="23.3934" width="0" layer="19" extent="1-1"/>
-<wire x1="85.725" y1="66.5734" x2="95.885" y2="48.7934" width="0" layer="19" extent="1-1"/>
 </signal>
 <signal name="UP_DOWN_CLK">
@@
 </signal>
 <signal name="!OUT+">
-<contactref element="U9" pad="3"/>
 <contactref element="U2" pad="12"/>
 <contactref element="U18" pad="2"/>
 <contactref element="U19" pad="1"/>
+<contactref element="U9" pad="3"/>
 <wire x1="76.2" y1="42.6466" x2="81.28" y2="79.2734" width="0" layer="19" extent="1-1"/>
 <wire x1="95.25" y1="17.2466" x2="76.2" y2="42.6466" width="0" layer="19" extent="1-1"/>
@@
 <contactref element="U12" pad="1"/>
 <contactref element="U12" pad="14"/>
-<contactref element="U9" pad="2"/>
 <contactref element="U19" pad="8"/>
 <contactref element="U9" pad="12"/>
+<contactref element="U9" pad="2"/>
 <wire x1="74.93" y1="42.6466" x2="76.2" y2="48.7934" width="0" layer="19" extent="1-1"/>
 <wire x1="52.705" y1="36.0934" x2="74.93" y2="42.6466" width="0" layer="19" extent="1-1"/>
@@
 <wire x1="85.09" y1="17.2466" x2="99.06" y2="17.2466" width="0" layer="19" extent="1-1"/>
 </signal>
-<signal name="N$27">
+<signal name="U13-13">
 <contactref element="U18" pad="12"/>
 <contactref element="U13" pad="13"/>
 <contactref element="U17" pad="12"/>
 <contactref element="U18" pad="6"/>
+<contactref element="U14" pad="8"/>
+<wire x1="96.52" y1="23.3934" x2="96.52" y2="36.0934" width="0" layer="19" extent="1-1"/>
 <wire x1="100.33" y1="17.2466" x2="96.52" y2="23.3934" width="0" layer="19" extent="1-1"/>
 <wire x1="81.28" y1="23.3934" x2="96.52" y2="23.3934" width="0" layer="19" extent="1-1"/>
@@
 <contactref element="R6" pad="2"/>
 <contactref element="R3" pad="2"/>
-<contactref element="U18" pad="8"/>
 <contactref element="U14" pad="6"/>
 <contactref element="U13" pad="1"/>
+<contactref element="U18" pad="8"/>
 <wire x1="95.25" y1="29.9466" x2="101.6" y2="23.3934" width="0" layer="19" extent="1-1"/>
 <wire x1="73.66" y1="29.9466" x2="95.25" y2="29.9466" width="0" layer="19" extent="1-1"/>
@@
 </signal>
 <signal name="!OUT-">
-<contactref element="U9" pad="11"/>
 <contactref element="U2" pad="2"/>
 <contactref element="U18" pad="1"/>
 <contactref element="U19" pad="13"/>
+<contactref element="U9" pad="11"/>
+<contactref element="U3" pad="3"/>
+<wire x1="80.01" y1="73.1266" x2="96.52" y2="73.1266" width="0" layer="19" extent="1-1"/>
 <wire x1="77.47" y1="48.7934" x2="80.01" y2="73.1266" width="0" layer="19" extent="1-1"/>
 <wire x1="93.98" y1="17.2466" x2="77.47" y2="48.7934" width="0" layer="19" extent="1-1"/>
@@
 <wire x1="53.34" y1="42.6466" x2="54.61" y2="48.7934" width="0" layer="19" extent="1-1"/>
 </signal>
+<signal name="U14-1">
+<contactref element="U19" pad="9"/>
+<contactref element="U14" pad="1"/>
+<contactref element="U19" pad="4"/>
+<wire x1="85.09" y1="10.6934" x2="88.9" y2="29.9466" width="0" layer="19" extent="1-1"/>
+<wire x1="82.55" y1="4.5466" x2="85.09" y2="10.6934" width="0" layer="19" extent="1-1"/>
+</signal>
+<signal name="N$25">
+<contactref element="U19" pad="10"/>
+<contactref element="U19" pad="5"/>
+<wire x1="83.82" y1="4.5466" x2="83.82" y2="10.6934" width="0" layer="19" extent="1-1"/>
+</signal>
+<signal name="U6-5">
+<contactref element="U3" pad="1"/>
+<contactref element="U3" pad="2"/>
+<contactref element="U6" pad="5"/>
+<contactref element="U6" pad="6"/>
+<contactref element="U10" pad="7"/>
+<wire x1="95.25" y1="73.1266" x2="93.98" y2="73.1266" width="0" layer="19" extent="1-1"/>
+<wire x1="99.06" y1="60.4266" x2="95.25" y2="73.1266" width="0" layer="19" extent="1-1"/>
+<wire x1="100.33" y1="60.4266" x2="99.06" y2="60.4266" width="0" layer="19" extent="1-1"/>
+<wire x1="95.885" y1="42.6466" x2="99.06" y2="60.4266" width="0" layer="19" extent="1-1"/>
+</signal>
+<signal name="U4-3">
+<contactref element="U3" pad="5"/>
+<contactref element="U4" pad="3"/>
+<wire x1="53.34" y1="57.8866" x2="99.06" y2="73.1266" width="0" layer="19" extent="1-1"/>
+</signal>
+<signal name="U5-7">
+<contactref element="U4" pad="1"/>
+<contactref element="U4" pad="2"/>
+<contactref element="U5" pad="7"/>
+<contactref element="U10" pad="5"/>
+<wire x1="93.345" y1="42.6466" x2="85.725" y2="60.4266" width="0" layer="19" extent="1-1"/>
+<wire x1="52.07" y1="57.8866" x2="85.725" y2="60.4266" width="0" layer="19" extent="1-1"/>
+<wire x1="50.8" y1="57.8866" x2="52.07" y2="57.8866" width="0" layer="19" extent="1-1"/>
+</signal>
+<signal name="U17-2">
+<contactref element="U2" pad="4"/>
+<contactref element="U17" pad="2"/>
+<contactref element="U17" pad="4"/>
+<contactref element="U17" pad="3"/>
+<wire x1="82.55" y1="17.2466" x2="82.55" y2="73.1266" width="0" layer="19" extent="1-1"/>
+<wire x1="81.28" y1="17.2466" x2="82.55" y2="17.2466" width="0" layer="19" extent="1-1"/>
+<wire x1="80.01" y1="17.2466" x2="81.28" y2="17.2466" width="0" layer="19" extent="1-1"/>
+</signal>
+<signal name="U13-12">
+<contactref element="U17" pad="1"/>
+<contactref element="U13" pad="12"/>
+<wire x1="78.74" y1="17.2466" x2="76.2" y2="36.0934" width="0" layer="19" extent="1-1"/>
+</signal>
+<signal name="U9-4">
+<contactref element="U17" pad="8"/>
+<contactref element="U9" pad="4"/>
+<wire x1="86.36" y1="23.3934" x2="77.47" y2="42.6466" width="0" layer="19" extent="1-1"/>
+</signal>
+<signal name="U13-3">
+<contactref element="U17" pad="9"/>
+<contactref element="U13" pad="3"/>
+<wire x1="76.2" y1="29.9466" x2="85.09" y2="23.3934" width="0" layer="19" extent="1-1"/>
+</signal>
+<signal name="U3-6">
+<contactref element="U3" pad="8"/>
+<contactref element="U6" pad="8"/>
+<contactref element="U6" pad="9"/>
+<contactref element="U3" pad="6"/>
+<wire x1="100.33" y1="73.1266" x2="101.6" y2="79.2734" width="0" layer="19" extent="1-1"/>
+<wire x1="100.33" y1="66.5734" x2="100.33" y2="73.1266" width="0" layer="19" extent="1-1"/>
+<wire x1="101.6" y1="66.5734" x2="100.33" y2="66.5734" width="0" layer="19" extent="1-1"/>
+</signal>
+<signal name="N$14">
+<contactref element="U18" pad="11"/>
+<contactref element="U17" pad="5"/>
+<wire x1="83.82" y1="17.2466" x2="97.79" y2="23.3934" width="0" layer="19" extent="1-1"/>
+</signal>
 </signals>
