File: bc29.brd (EAGLE design)
At the start: 116.8 x 86.4 mm, 107 parts, among them IC1 TSC900BIJA, IC10 MC14516B, IC11 CD4070B, IC12 MC14516B, IC13 CD4013, IC14 CD4023, IC15 CD4013B, IC16 MC14073B, IC17 CD4070B, IC18 LP2951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

Commit message: Incorperate display module knowldge
Parts:
- removed J1: 2520-5, con-3m:PAK100/2500-5-20
- added J2: 2520-5, con-3m:PAK100/2500-5-20
Connections:
- removed net !DOWN: IC10.10, IC11.10, IC11.13, IC12.10, IC14.4, IC16.11, IC5.6, J1.1
- removed net !LCD_RESET: IC3.4, J1.17
- removed net !UP_DOWN_CLK: IC11.3, IC14.11, IC9.6, J1.15
- removed net AH_NEGATIVE_LCD: IC11.9, IC8.9, IC9.11, IC9.2, J1.18
- removed net LCD-13: IC14.9, IC19.5, J1.13
- removed net LCD-16: IC15.5, IC9.12, IC9.3, J1.16
- removed net LCD-3: C20.1, IC19.6, J1.3
- removed net LCD_45_HZ: IC17.12, IC17.2, IC17.5, IC17.9, J1.19
- removed net V_F_OUT: D7.C, E1.-, J1.20
- new net !IN_LED: IC11.9, IC8.9, IC9.11, IC9.2, J2.18
- new net !LCD_COUNTER_BACKPLANE: IC17.12, IC17.2, IC17.5, IC17.9, J2.19
- new net !LCD_COUNTER_CARRY: C20.1, IC19.6, J2.3
- new net !LCD_COUNTER_CLK: IC11.3, IC14.11, IC9.6, J2.15
- new net !LCD_COUNTER_RESET: IC3.4, J2.17
- new net !OUT_LED: IC15.5, IC9.12, IC9.3, J2.16
- new net LCD_COUNTER_BLANK: IC16.10, J2.9
- new net LCD_COUNTER_ENABLE: IC14.9, IC19.5, J2.13
- new net LCD_COUNTER_UP: IC10.10, IC11.10, IC11.13, IC12.10, IC14.4, IC16.11, IC5.6, J2.1
- new net LED_ANODE: D7.C, E1.-, J2.20
- net +5V: now also J2.14; no longer J1.14
- net 12+: now also J2.4; no longer J1.4
- net 12-: now also J2.2; no longer J1.2
- net GND: now also J2.5; no longer J1.5
- net LCD_COLON: now also J2.11; no longer J1.11
- net LCD_DECIMAL_POINT: now also J2.7; no longer J1.7
- net LCD_MINUS_SIGN: now also J2.8; no longer J1.8
- net LCD_ONE_MSD: now also J2.10; no longer J1.10
- net OVER_FLOW_UP: no longer IC16.10, J1.9

Commit message: Move things around. Update png files
Connections:
- net IC15-12 renamed !OVER_FLOW
- net IC16-2 renamed ENABLE_OR_NOT_CARRY
- net GND: now also IC13.4
Changed lines of the file:
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@@
 <contactref element="R17" pad="2"/>
 <contactref element="J2" pad="5"/>
-<wire x1="73.66" y1="74.93" x2="72.52" y2="81.28" width="0" layer="19" extent="1-1"/>
-<wire x1="68.58" y1="74.93" x2="73.66" y2="74.93" width="0" layer="19" extent="1-1"/>
-<wire x1="66.47" y1="72.39" x2="68.58" y2="74.93" width="0" layer="19" extent="1-1"/>
-<wire x1="59.63" y1="75.565" x2="66.47" y2="72.39" width="0" layer="19" extent="1-1"/>
-<wire x1="54.29" y1="73.66" x2="59.63" y2="75.565" width="0" layer="19" extent="1-1"/>
-<wire x1="63.18" y1="81.28" x2="59.63" y2="75.565" width="0" layer="19" extent="1-1"/>
-<wire x1="81.915" y1="66.5734" x2="73.66" y2="74.93" width="0" layer="19" extent="1-1"/>
-<wire x1="83.185" y1="66.5734" x2="81.915" y2="66.5734" width="0" layer="19" extent="1-1"/>
-<wire x1="81.915" y1="60.4266" x2="81.915" y2="66.5734" width="0" layer="19" extent="1-1"/>
-<wire x1="80.645" y1="60.4266" x2="81.915" y2="60.4266" width="0" layer="19" extent="1-1"/>
-<wire x1="78.105" y1="60.4266" x2="80.645" y2="60.4266" width="0" layer="19" extent="1-1"/>
-<wire x1="92.075" y1="48.7934" x2="81.915" y2="60.4266" width="0" layer="19" extent="1-1"/>
-<wire x1="93.345" y1="48.7934" x2="92.075" y2="48.7934" width="0" layer="19" extent="1-1"/>
-<wire x1="96.52" y1="51.64" x2="93.345" y2="48.7934" width="0" layer="19" extent="1-1"/>
+<contactref element="IC13" pad="4"/>
+<wire x1="96.52" y1="51.64" x2="97.79" y2="60.4266" width="0" layer="19" extent="1-1"/>
+<wire x1="93.345" y1="48.7934" x2="96.52" y2="51.64" width="0" layer="19" extent="1-1"/>
+<wire x1="92.075" y1="48.7934" x2="93.345" y2="48.7934" width="0" layer="19" extent="1-1"/>
 <wire x1="101.6" y1="48.26" x2="96.52" y2="51.64" width="0" layer="19" extent="1-1"/>
 <wire x1="92.075" y1="42.6466" x2="92.075" y2="48.7934" width="0" layer="19" extent="1-1"/>
@@
 <wire x1="31.75" y1="12.27" x2="35.56" y2="12.27" width="0" layer="19" extent="1-1"/>
 <wire x1="22.86" y1="10.16" x2="31.75" y2="12.27" width="0" layer="19" extent="1-1"/>
+<wire x1="81.915" y1="60.4266" x2="92.075" y2="48.7934" width="0" layer="19" extent="1-1"/>
+<wire x1="80.645" y1="60.4266" x2="81.915" y2="60.4266" width="0" layer="19" extent="1-1"/>
+<wire x1="78.105" y1="60.4266" x2="80.645" y2="60.4266" width="0" layer="19" extent="1-1"/>
+<wire x1="81.915" y1="66.5734" x2="81.915" y2="60.4266" width="0" layer="19" extent="1-1"/>
+<wire x1="83.185" y1="66.5734" x2="81.915" y2="66.5734" width="0" layer="19" extent="1-1"/>
+<wire x1="73.66" y1="74.93" x2="81.915" y2="66.5734" width="0" layer="19" extent="1-1"/>
+<wire x1="68.58" y1="74.93" x2="73.66" y2="74.93" width="0" layer="19" extent="1-1"/>
+<wire x1="66.47" y1="72.39" x2="68.58" y2="74.93" width="0" layer="19" extent="1-1"/>
+<wire x1="72.52" y1="81.28" x2="73.66" y2="74.93" width="0" layer="19" extent="1-1"/>
+<wire x1="59.63" y1="75.565" x2="66.47" y2="72.39" width="0" layer="19" extent="1-1"/>
+<wire x1="54.29" y1="73.66" x2="59.63" y2="75.565" width="0" layer="19" extent="1-1"/>
+<wire x1="63.18" y1="81.28" x2="59.63" y2="75.565" width="0" layer="19" extent="1-1"/>
 <wire x1="42.23" y1="60.96" x2="54.29" y2="73.66" width="0" layer="19" extent="1-1"/>
 <wire x1="34.29" y1="55.94" x2="42.23" y2="60.96" width="0" layer="19" extent="1-1"/>
@@
 <wire x1="50.8" y1="57.8866" x2="52.07" y2="57.8866" width="0" layer="19" extent="1-1"/>
 </signal>
-<signal name="IC16-2">
+<signal name="ENABLE_OR_NOT_CARRY">
 <contactref element="IC19" pad="4"/>
 <contactref element="IC16" pad="2"/>
@@
 <wire x1="80.01" y1="17.2466" x2="81.28" y2="17.2466" width="0" layer="19" extent="1-1"/>
 </signal>
-<signal name="IC15-12">
+<signal name="!OVER_FLOW">
 <contactref element="IC16" pad="1"/>
 <contactref element="IC15" pad="12"/>
@@
 <signal name="LCD_COUNTER_ENABLE">
 <contactref element="J2" pad="13"/>
+<contactref element="IC19" pad="5"/>
 <contactref element="IC14" pad="9"/>
-<contactref element="IC19" pad="5"/>
 <wire x1="83.82" y1="73.1266" x2="100.33" y2="79.2734" width="0" layer="19" extent="1-1"/>
 <wire x1="20.955" y1="-17.78" x2="83.82" y2="73.1266" width="0" layer="19" extent="1-1"/>

Commit message: Clean up net names
Connections:
- net !LCD_COUNTER_BACKPLANE renamed LCD_COUNTER_BACKPLANE
- net !LCD_COUNTER_CLK renamed LCD_COUNTER_CLK
- removed net IC17-1: IC9.4, IC9.9
- net COLON_ON: now also IC9.4, IC9.9
Changed lines of the file:
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@@
 <?xml version="1.0" encoding="utf-8"?>
 <!DOCTYPE eagle SYSTEM "eagle.dtd">
-<eagle version="7.1.0">
+<eagle version="7.2.0">
 <drawing>
 <settings>
@@
 <wire x1="53.34" y1="42.6466" x2="54.61" y2="48.7934" width="0" layer="19" extent="1-1"/>
 </signal>
-<signal name="IC17-1">
-<contactref element="IC9" pad="9"/>
-<contactref element="IC9" pad="4"/>
-<wire x1="82.55" y1="4.5466" x2="85.09" y2="10.6934" width="0" layer="19" extent="1-1"/>
-</signal>
 <signal name="N$25">
 <contactref element="IC9" pad="10"/>
@@
 <signal name="COLON_ON">
 <contactref element="IC17" pad="1"/>
+<contactref element="IC9" pad="9"/>
+<contactref element="IC9" pad="4"/>
+<wire x1="85.09" y1="10.6934" x2="88.9" y2="29.9466" width="0" layer="19" extent="1-1"/>
+<wire x1="82.55" y1="4.5466" x2="85.09" y2="10.6934" width="0" layer="19" extent="1-1"/>
 </signal>
 <signal name="!LCD_COUNTER_CARRY">
@@
 <wire x1="26.035" y1="-17.78" x2="34.925" y2="37.5666" width="0" layer="19" extent="1-1"/>
 </signal>
-<signal name="!LCD_COUNTER_BACKPLANE">
+<signal name="LCD_COUNTER_BACKPLANE">
 <contactref element="J2" pad="19"/>
 <contactref element="IC17" pad="2"/>
@@
 <wire x1="28.575" y1="-15.24" x2="90.17" y2="52.07" width="0" layer="19" extent="1-1"/>
 </signal>
-<signal name="!LCD_COUNTER_CLK">
+<signal name="LCD_COUNTER_CLK">
 <contactref element="J2" pad="15"/>
 <contactref element="IC11" pad="3"/>

Commit message: Clean up some net names
Connections:
- net N$20 renamed !CHARGE
- net N$21 renamed !DISCHARGE
- net N$53 renamed D_CHARGE
- net N$55 renamed NEG_COMPARATOR
- net N$56 renamed POS_COMPARATOR
- net N$57 renamed D_DISCHARGE
- net OUT renamed OP_AMP__OUT
Changed lines of the file:
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@@
 <wire x1="48.26" y1="3.68" x2="46.99" y2="19.05" width="0" layer="19" extent="1-1"/>
 </signal>
-<signal name="OUT">
+<signal name="OP_AMP__OUT">
 <contactref element="IC1" pad="6"/>
 <contactref element="C1" pad="2"/>
@@
 <wire x1="36.83" y1="50.74" x2="31.75" y2="55.94" width="0" layer="19" extent="1-1"/>
 </signal>
-<signal name="N$55">
+<signal name="NEG_COMPARATOR">
 <contactref element="IC2" pad="8"/>
 <contactref element="R16" pad="1"/>
 <wire x1="39.37" y1="55.94" x2="42.23" y2="55.88" width="0" layer="19" extent="1-1"/>
 </signal>
-<signal name="N$56">
+<signal name="POS_COMPARATOR">
 <contactref element="IC2" pad="1"/>
 <contactref element="R15" pad="1"/>
@@
 <wire x1="20" y1="59.69" x2="54.29" y2="53.34" width="0" layer="19" extent="1-1"/>
 </signal>
-<signal name="N$53">
+<signal name="D_CHARGE">
 <contactref element="R15" pad="2"/>
 <contactref element="IC4" pad="5"/>
 <wire x1="44.13" y1="52.07" x2="55.88" y2="42.6466" width="0" layer="19" extent="1-1"/>
 </signal>
-<signal name="N$57">
+<signal name="D_DISCHARGE">
 <contactref element="R16" pad="2"/>
 <contactref element="IC4" pad="9"/>
@@
 <signal name="1_024KHZ">
 <contactref element="IC6" pad="5"/>
+<contactref element="IC4" pad="8"/>
 <contactref element="IC8" pad="12"/>
 <contactref element="IC4" pad="6"/>
-<contactref element="IC4" pad="8"/>
 <wire x1="58.42" y1="48.7934" x2="53.34" y2="64.0334" width="0" layer="19" extent="1-1"/>
 <wire x1="57.15" y1="42.6466" x2="58.42" y2="48.7934" width="0" layer="19" extent="1-1"/>
@@
 <wire x1="97.79" y1="17.2466" x2="80.01" y2="36.0934" width="0" layer="19" extent="1-1"/>
 </signal>
-<signal name="N$20">
+<signal name="!CHARGE">
 <contactref element="IC5" pad="8"/>
 <contactref element="IC4" pad="2"/>
 <wire x1="52.07" y1="42.6466" x2="81.28" y2="48.7934" width="0" layer="19" extent="1-1"/>
 </signal>
-<signal name="N$21">
+<signal name="!DISCHARGE">
 <contactref element="IC4" pad="12"/>
 <contactref element="IC5" pad="9"/>
@@
 </signal>
 <signal name="!1_024KHZ">
-<contactref element="IC4" pad="3"/>
 <contactref element="IC4" pad="11"/>
 <contactref element="IC8" pad="11"/>
+<contactref element="IC4" pad="3"/>
 <wire x1="54.61" y1="48.7934" x2="54.61" y2="64.0334" width="0" layer="19" extent="1-1"/>
 <wire x1="53.34" y1="42.6466" x2="54.61" y2="48.7934" width="0" layer="19" extent="1-1"/>

Commit message: Rference files on Yahoo Solectria_EV site
Parts:
- moved J2 101.1 mm to (99.7, 41.9), turned to 270 degrees
- moved C20 4.58 mm to (97.8, 53.3), turned to 90 degrees
