File: bc29.sch (EAGLE design)
At the start: 67 parts, among them IC1 LP2951D, IC10 TLC27L41, IC11 4001D, IC2 HCF4520, IC3 4053D, IC4 4093D, IC5 4013D, IC6 4013D, IC8 Teledyne TSC900BIJA, IC9 4060D, Q1 IRF740, X1 32KHz, X2 2520-5

Commit message: Complete board silk screen. Update schematic to match
Parts:
- removed IC1: LP2951D, linear:LP2951D
- removed IC10: TLC27L41, linear:TLC274D
- removed IC11: 4001D, 40xx:4001D
- removed IC2: HCF4520, 45xx:4520D
- removed IC3: 4053D, 40xx:4053D
- removed IC4: 4093D, 40xx:4093D
- removed IC5, IC6: 4013D, 40xx:4013D
- removed IC8: Teledyne TSC900BIJA, ic-package:DIL8S
- removed IC9: 4060D, 40xx:4060D
- removed SL1: (no value), con-amp-quick:M12
- removed X2: 2520-5, con-3m:2520-5
- added C18: (no value), rcl:C-EU050-045X075
- added C19, C20, C21, C22, C23, C24, C25, C27, C28: (no value), rcl:C-EUC0805
- added D11: 1n4148, diode:DIODE-MINIMELF
- added J1: 2520-5, con-3m:2520-5
- added JP10, JP11, JP12, JP2, JP3, JP4, JP5, JP6, JP7, JP8, JP9: (no value), pinhead:PINHD-1X1
- added JP13: (no value), pinhead:PINHD-1X12
- added R13: 3K, rcl:R-EU_M0805
- added R14: 1M, rcl:R-EU_M0805
- added R27: 47, rcl:R-EU_M0805
- added R28: 10M, rcl:R-EU_M0805
- added R29: 330K, rcl:R-EU_M0805
- added R30, R32: 1K, rcl:R-EU_M0805
- added R31: 10K, rcl:R-EU_M0805
- added RX: OPEN, rcl:R-EU_0207/10
- added U1: LP2951, linear:LP2951D
- added U10, U5: MC14516B, 45xx:4516D
- added U11: CD4053B, 40xx:4053D
- added U12: HCF4520, 45xx:4520D
- added U13, U8: CD4013B, 40xx:4013D
- added U14, U18: CD4070B, 40xx:4070D
- added U15: TSC900BIJA, linear:2CMPN
- added U16: CD4060B, 40xx:4060D
- added U17: MC14073B, 40xx:4073D
- added U19, U9: CD4001B, 40xx:4001D
- added U2: CD4081, 40xx:4081D
- added U3: CD4023, 40xx:4023D
- added U4: CD4093B, 40xx:4093D
- added U6: CD4013, 40xx:4013D
- added U7: TLC27L41, linear:TLC274D
- C1: device rcl:C-EU050-025X075 -> rcl:C-EU050-024X044
- C10, C11: value Poly -> (none); device rcl:C-EU050-025X075 -> rcl:C-EUC1206
- C12, C13, C14, C15, C8, C9: device rcl:C-EU050-025X075 -> rcl:C-EUC1206
- C16: value 10uF 63V -> (none); device rcl:CPOL-EUB45181A -> rcl:C-EUC1206
- C17: device rcl:C-EU050-025X075 -> rcl:C-EU050-045X075
- C2, C3: value (none) -> 47uf 25V; device rcl:C-EU050-025X075 -> rcl:CPOL-EUE2.5-5
- C4: value 47uF 25V -> 47uf 25V; device rcl:CPOL-EUB45181A -> rcl:CPOL-EUE2.5-5
- C5, C6: value 47uF 25V -> 10uF 63V; device rcl:CPOL-EUB45181A -> rcl:CPOL-EUE2.5-5
- C7: value (none) -> 10uF 63V; device rcl:C-EU050-025X075 -> rcl:CPOL-EUE2.5-5
- D1: value 1N4148 -> V674; device diode:1N4148DO35-7 -> diode:DIODE-SOD80C
- D10, D8, D9: value PMLL4150 -> 1n4148; device diode:PMLL4150 -> diode:DIODE-MINIMELF
- D2, D4: device diode:1N4148DO35-7 -> diode:DIODE-MINIMELF
- D3, D5: value 1N4148 -> ZENER?; device diode:1N4148DO35-7 -> diode:DIODE-MINIMELF
- D6: value 1N4148 -> 1n4148; device diode:1N4148DO35-7 -> diode:DIODE-MINIMELF
- D7: value PMLL4150 -> 1N4148; device diode:PMLL4150 -> diode:DIODE-MINIMELF
- JP1: device pinhead:PINHD-1X12 -> pinhead:PINHD-1X1
- R1: value 1M -> 20K; device rcl:R-EU_0207/10 -> rcl:R-EU_M0805
- R10: device rcl:R-EU_0207/10 -> rcl:R-EU_M0805
- R11: value (none) -> 1M; device rcl:R-EU_0207/10 -> rcl:R-EU_M0805
- R12: value 3K -> 1M; device rcl:R-EU_0207/10 -> rcl:R-EU_M0805
- R15: value 10M -> 1M; device rcl:R-EU_0207/10 -> rcl:R-EU_M0805
- R16: value 330K -> 100K; device rcl:R-EU_0207/10 -> rcl:R-EU_M0805
- R17: value 1M -> 100K; device rcl:R-EU_0207/10 -> rcl:R-EU_M0805
- R18: value 1M -> 300; device rcl:R-EU_0207/10 -> rcl:R-EU_M0805
- R19: value 330K -> 300; device rcl:R-EU_0207/10 -> rcl:R-EU_M0805
- R2: value 300 -> 20K; device rcl:R-EU_0207/10 -> rcl:R-EU_M0805
- R20: value 330K -> 2K; device rcl:R-EU_0207/10 -> rcl:R-EU_M0805
- R21: value 330K -> 130K
- R22: value 2K -> 130K
- R23: value 2K -> 4.70K
- R24: value 2K -> 8.20K
- R25: value 20K -> 620; device rcl:R-EU_0207/10 -> rcl:R-EU_M0805
- R26: value 1K -> 47; device rcl:R-EU_0207/10 -> rcl:R-EU_M0805
- R3: value 620 -> 2K; device rcl:R-EU_0207/10 -> rcl:R-EU_M0805
- R4: value 300 -> 2K; device rcl:R-EU_0207/10 -> rcl:R-EU_M0805
- R5: value 47 -> 2K; device rcl:R-EU_0207/10 -> rcl:R-EU_M0805
- R6: value 47 -> 100K; device rcl:R-EU_0207/10 -> rcl:R-EU_M0805
- R7, R8: value 130K -> 330K; device rcl:R-EU_0207/10 -> rcl:R-EU_M0805
- R9: value 110K -> 330K; device rcl:R-EU_0207/10 -> rcl:R-EU_M0805
- X1: value 32KHz -> 32.768KHz; device crystal:FC-12M -> crystal:CRYSTALTC26H
Connections:
- removed net +12V: D9.A, IC10P.V+, IC3A.Y, R18.1, R5.2
- removed net 12V+: JP1.11, SL1.11, X2-4.KL
- removed net 12V-: JP1.12, SL1.12, X2-2.KL
- removed net 2KHZ: C6.+, IC9A.Q4
- removed net 32_47KHZ: IC9A.P0
- removed net N$1: D10.A, F1.2, R10.2
- removed net N$10: C3.1, IC8.4, R6.1
- removed net N$11: C7.2, IC8.1
- removed net N$12: C8.2, C9.2, IC10A.-IN, IC8.6
- removed net N$2: R1.2, R10.1
- removed net N$3: C10.1, D5.A, D6.C, IC8.3, R3.1
- removed net N$4: C11.1, R2.2, R4.1
- removed net N$5: C12.1, C8.1, C9.1, D3.C, D4.A, IC8.2, R11.2, R4.2, R7.2
- removed net N$6: C1.2, IC8.8
- removed net N$7: C2.2, IC8.7, R5.1
- removed net N$8: C12.2, IC3A.Y0, R8.2
- removed net N$9: C6.-, D1.C, D2.A
- new net -1V25: C20.2, C21.1, R7.2, R8.1, U7C.-IN
- new net 0V0: C21.2, R8.2, R9.1, U7D.-IN
- new net 12+: J1-4.KL, JP11.1, JP13.11
- new net 12-: J1-2.KL, JP12.1, JP13.12
- new net 13V5: C5.+, D2.A, Q1.S, U1.IN
- new net 1V25: C22.2, R12.1, R9.2, U7A.+IN
- new net 1_024KHZ: U16A.Q5
- new net 1_031KHZ: U8A.CLK, U8B.CLK
- new net 2_048KHZ: C3.+, U16A.Q4
- new net 32_768KHZ: R28.1, R29.1, U16A.!P0
- new net 4HZ: U12A.EN, U16A.Q13
- new net DRAIN: D1.C, Q1.D
- new net FUSED_BATT+: D1.A, F1.2, R14.2
- new net GATE: C23.1, D2.C, D3.C, Q1.G, R15.2
- new net LCD-20: C6.-, D5.C, J1-20.KL
- new net N$14: J1-10.KL, U14C.O
- new net N$16: J1-8.KL, U14B.O
- new net N$39: C27.2, R29.2, X1.1
- new net N$40: C28.2, R28.2, U16A.P1, X1.2
- new net N$41: C13.1, U15.CMP1
- new net N$42: R21.1, R22.2
- new net N$43: C14.1, U15.CMP2
- new net N$44: U1.FB, U1.VOTAB
- new net N$45: R23.1, R24.2
- new net N$46: R13.1, U11A.X
- new net N$47: R13.2, U7B.-IN, U7B.OUT
- new net N$48: R16.1, U4C.O
- new net N$49: R17.2, U13A.S
- new net N$51: C19.1, R1.2, R6.1
- new net N$52: U10A.CLK, U5A.CLK
- new net N$53: R11.2, U8A.D
- new net N$54: C6.+, R32.1
- new net N$55: R10.1, U7C.OUT
- new net N$56: R11.1, U7A.OUT
- new net N$57: R10.2, U8B.D
- new net N$60: U19C.I0, U9A.I1
- new net RESET_R: C7.+, C9.1, R16.2, R2.2, U4B.I0, U4B.I1
- new net U8-1: U11A.B, U8A.Q, U9A.I0
- new net U8-13: U11A.A, U8B.Q
- new net U8-SET: C25.1, R17.1, U4D.I0, U8A.S, U8B.S
- net !RESET: now also U4B.O; no longer IC3A.C, IC4B.O, IC5A.R, IC6B.R
- net +5V: now also C2.+, C24.1, C8.1, D3.A, D4.C, J1-14.KL, R12.2, R26.2, U1.OUT, U1.SENSE, U11A.Y, U11A.Z0, U4D.I1, U7P.V+; no longer C15.2, C4.+, D8.C, IC1.OUT, IC1.SENSE
- net +BATT: now also JP13.1; no longer SL1.1
- net -2V5: now also C20.1, R7.1, U7B.+IN, U7D.OUT; no longer IC10B.+IN
- net -4V: now also C4.-, D11.A; no longer C5.-, D1.A, IC10P.V-
- net -5V: now also C16.1, R27.1, U7P.V-; no longer R6.2
- net AH_NEGATIVE: now also JP13.8, JP8.1, R3.1; no longer JP1.8, R23.1, SL1.8
- net GND: now also C1.2, C12.2, C13.2, C14.2, C15.2, C16.2, C17.2, C18.2, C19.2, C2.-, C22.1, C23.2, C24.2, C27.1, C28.1, C4.+, C5.-, C7.-, C8.2, C9.2, D10.C, D4.A, D7.C, D9.C, J1-5.KL, JP13.2, JP2.1, R30.2, U1.GND, U11A.INH, U11A.Z1, U16A.RES, U7D.+IN, U8A.R, U8B.R; no longer C1.1, C10.2, C11.2, C13.1, C14.1, C16.-, C17.1, C2.1, C3.2, C4.-, C5.+, C7.1, D2.C, D3.A, D4.C, D5.C, IC1.GND, IC3A.INH, IC9A.RES, JP1.2, R26.2, SL1.2, X2-3.KL
- net GND1K: now also JP13.6, JP6.1, R30.1; no longer JP1.6, R26.1, SL1.6
- net N$13: now also C1.1, J1-3.KL, U2B.O; no longer IC3A.X0, R9.2
- net N$15: now also J1-1.KL, U18C.O; no longer C13.2, IC9A.P1, R15.1, X1.2
- net N$17: now also J1-7.KL, U14D.O; no longer R11.1, R9.1
- net N$18: now also J1-9.KL, U17C.O, U5A.CIN; no longer R7.1, R8.1
- net N$19: now also J1-11.KL, U14A.O; no longer IC10B.-IN, IC10B.OUT, R12.2
- net N$20: now also J1-13.KL, U3A.O; no longer IC3A.X, R12.1
- net N$21: now also J1-15.KL, U18A.O, U3C.I0; no longer C14.2, R16.1, X1.1
- net N$22: now also J1-17.KL, U11A.Z; no longer IC9A.!P0, R15.2, R16.2
- net N$23: now also J1-19.KL, U14A.I1, U14B.I0, U14C.I1, U14D.I0; no longer IC10A.+IN, R18.2, R19.2
- net N$24: now also C25.2, U19C.O; no longer IC10A.OUT, R17.2
- net N$25: now also D5.A, U10A.P1; no longer R19.1, R20.2
- net N$26: now also J1-18.KL, U18C.I1, U4C.I1; no longer R20.1, R21.2
- net N$27: now also C18.1, R18.2, R19.1; no longer IC2A.EN, IC9A.Q13
- net N$28: now also J1-16.KL, U19A.O; no longer IC10D.OUT, R21.1
- net N$29: now also R14.1, R15.1; no longer D10.C, Q1.D
- net N$30: now also C10.1, C11.1, D6.C, D7.A, R19.2, R20.1, R21.2, R23.2, R31.1, RX.2, U15.-IN; no longer C15.1, IC1.FB
- net N$31: now also C15.1, R26.1, U15.V+; no longer IC3A.A, IC5B.Q
- net N$32: now also R32.2, U5A.Q3; no longer IC10D.+IN, IC3A.Z1
- net N$33: now also C12.1, R27.2, U15.V-; no longer IC11A.I0, IC3A.B, IC5A.Q
- net N$34: now also C10.2, C11.2, U15.OUT, U7A.-IN, U7C.+IN; no longer IC3A.Z
- net N$35: now also R20.2, R24.1, RX.1, U11A.X0; no longer IC5A.D, R17.1
- net N$36: now also C17.1, D8.C, D9.A, U15.+IN; no longer IC4B.I0, IC4B.I1
- net N$37: now also R22.1, R31.2, U11A.Y0; no longer C17.2, D7.C, D9.C, Q1.G, R1.1
- net N$38: now also C3.-, D10.A, D11.C; no longer C16.+, D7.A, IC1.IN, Q1.S
- net NAR: now also JP13.5, JP5.1, R1.1; no longer JP1.5, SL1.5
- net OUT+: now also JP13.9, JP9.1, R4.1; no longer JP1.9, R24.1, SL1.9
- net OUT-: now also JP10.1, JP13.10, R5.1; no longer JP1.10, R22.1, SL1.10
- net RESET: now also JP13.7, JP7.1, R2.1; no longer JP1.7, R25.1, SL1.7
- net SHUNT+: now also JP13.4, JP4.1, R18.1; no longer JP1.4, R2.1, SL1.4
- net SHUNT-: now also JP13.3, JP3.1, R25.1; no longer JP1.3, R3.2, SL1.3
Other:
- note added: "13.5VDC"
- note added: "4 Hz/A Charged"
- note added: "4 Hz/A Discharged"
- note added: "Backlight"
- note added: "Delta Sigma Converter"
- note added: "LCD"
- note added: "NO AUTO RESET"
- note added: "Resistor Trim"
- note removed: "Chopper-Stabilized Op Amp"
- moved on the sheet: C1, C10, C11, C12, C13, C14, C15, C17, C4, C5, C6, C8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

Commit message: Charge/discharge output
Connections:
- net NAR renamed !NAR
- net U8-1 renamed CHARGE
- removed net 1_031KHZ: U8A.CLK, U8B.CLK
- removed net U8-13: U11A.A, U8B.Q
- new net DISCHAR: U11A.A, U8B.Q, U9D.I1
- new net N$50: R5.2, U2A.O
- new net N$58: R4.2, U2D.O
- new net N$59: U2A.I1, U9D.O
- new net N$61: U2D.I0, U9A.O
- new net U13-1: R3.2, R6.2, U13A.Q
- net !RESET: now also JP13.7, JP7.1, R2.1; no longer U4B.O
- net +5V: now also U2A.I0, U2D.I1
- net 1_024KHZ: now also U8A.CLK, U8B.CLK
- net RESET: now also U4B.O; no longer JP13.7, JP7.1, R2.1
Other:
- note added: "Reference Voltage Generator"
- moved on the sheet: C19, C20, C21, C22, JP1, JP10, JP11, JP12, JP13, JP2, JP3, JP4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

Commit message: more charge/discharge
Connections:
- net DISCHAR renamed DISCHARGE
- net N$13 renamed LCD-3
- net N$14 renamed LCD-10
- net N$15 renamed LCD-1
- net N$16 renamed LCD-8
- net N$17 renamed LCD-7
- net N$18 renamed LCD-9
- net N$19 renamed LCD-11
- net N$20 renamed LCD-13
- net N$21 renamed LCD-15
- net N$22 renamed LCD-17
- net N$23 renamed LCD-19
- net N$26 renamed LCD-18
- net N$28 renamed LCD-16
- net N$30 renamed IN-
- net N$31 renamed VDD+
- net N$33 renamed VDD-
- net N$34 renamed OUT
- net N$36 renamed IN+
- net N$41 renamed CXA
- net N$43 renamed CXB
- net N$46 renamed -2V5_BUF_R
- net N$47 renamed -2V5_BUF
- net RESET: now also U13A.R, U13B.R, U5A.RES, U6B.R
Other:
- note added: "LCD Interface"
- moved on the sheet: C1, C25, C6, D5, J1-1, J1-10, J1-11, J1-12, J1-13, J1-14, J1-15, J1-16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

Commit message: Digital updates
Connections:
- net LCD-15 renamed !UP_DOWN_CLK
- net N$27 renamed SHUNT+FILTER
- net N$35 renamed X0
- net N$37 renamed Y0
- removed net LCD-1: J1-1.KL, U18C.O
- removed net N$25: D5.A, U10A.P1
- removed net N$52: U10A.CLK, U5A.CLK
- new net !DOWN: J1-1.KL, U10A.U/!D, U17C.I0, U18C.O, U18D.I1, U5A.U/!D, U9B.I1
- new net N$13: U10A.P3, U14D.I1
- new net N$14: U10A.CO, U6A.D, U6A.S
- new net N$15: U10A.RES
- new net N$16: U14B.I1, U18C.I0
- new net N$17: U10A.PE, U6A.!Q
- new net N$18: U3B.O, U6B.D, U6B.S
- new net N$19: U10A.CIN, U5A.CO
- new net UP_DOWN_CLK: U10A.CLK, U3C.O, U5A.CLK, U6A.CLK, U6B.CLK
- net +5V: now also U3C.I1, U3C.I2
- net GND: now also D5.A, U10A.P0, U10A.P1, U10A.P2, U5A.P0, U5A.P1, U5A.P2, U5A.P3, U5A.PE
- net RESET: now also U11A.C
Other:
- moved on the sheet: C10, C11, C12, C13, C14, C15, C16, C17, C18, C6, D5, D6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

Commit message: cleanup up/down counter
Connections:
- net LCD-18 renamed AH_NEGATIVE_LCD
- net N$50 renamed OUT-_R
- net N$58 renamed OUT+_R
- removed net N$49: R17.2, U13A.S
- removed net N$51: C19.1, R1.2, R6.1
- removed net N$59: U2A.I1, U9D.O
- removed net N$60: U19C.I0, U9A.I1
- removed net N$61: U2D.I0, U9A.O
- removed net U13-1: R3.2, R6.2, U13A.Q
- removed net U8-SET: C25.1, R17.1, U4D.I0, U8A.S, U8B.S
- new net !1_024KHZ: U4D.O, U8A.CLK, U8B.CLK
- new net !NAR_R: C19.1, R1.2, R6.1, U4C.I0
- new net !OUT+: U18A.I1, U19A.I0, U2D.I0, U9A.O
- new net !OUT-: U18A.I0, U19D.I1, U2A.I1, U9D.O
- new net AH_NEGATIVE_R: R3.2, R6.2, U13A.Q, U14B.I1, U18C.I0
- new net N$20: U8A.!Q, U9C.I0
- new net N$21: U8B.!Q, U9C.I1
- new net N$22: U19A.I1, U19D.O
- new net N$23: U12A.Q3, U12B.CLK
- new net N$26: U17B.O, U18B.I0
- new net N$27: U13B.Q, U17C.I1, U18B.I1, U18D.I0
- new net U12-14: U12A.CLK, U12B.Q3, U19C.I0, U9A.I1, U9D.I0
- net +5V: now also U10A.P3, U12B.EN, U14D.I1, U17C.I2
- net 1_024KHZ: now also U4D.I0, U8A.S, U8B.S; no longer U8A.CLK, U8B.CLK
- net GND: now also R17.2, U13A.S, U13B.S
- net LCD-16: now also U13A.D, U19D.I0
- net N$13: now also C25.2, U9C.O; no longer U10A.P3, U14D.I1
- net N$15: now also U6B.!Q
- net N$16: now also U13B.D, U18B.O; no longer U14B.I1, U18C.I0
- net N$24: now also C25.1, R17.1, U12A.RES, U12B.RES; no longer C25.2, U19C.O
- net UP_DOWN_CLK: now also U13B.CLK, U9B.I0
Other:
- moved on the sheet: C1, C19, C2, C20, C21, C22, C23, C24, C25, C27, C28, C3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

Commit message: cleanup random gates
Connections:
- removed net N$18: U3B.O, U6B.D, U6B.S
- removed net N$19: U10A.CIN, U5A.CO
- removed net N$27: U13B.Q, U17C.I1, U18B.I1, U18D.I0
- new net N$25: U19B.I0, U19C.O
- new net U13-12: U13B.!Q, U17A.I0
- new net U13-13: U13B.Q, U14C.I0, U17C.I1, U18B.I1, U18D.I0
- new net U13-3: U13A.CLK, U17A.O
- new net U14-1: U14A.I0, U19B.O, U19C.I1
- new net U17-2: U17A.I1, U17B.I0, U17B.I1, U2B.O
- new net U3-6: U3A.I2, U3B.O, U6B.D, U6B.S
- new net U4-3: U3B.I2, U4A.O
- new net U5-7: U10A.CIN, U4A.I0, U4A.I1, U5A.CO
- new net U6-5: U10A.CO, U3A.I0, U3A.I1, U6A.D, U6A.S
- new net U9-4: U17A.I2, U9B.O
- net !DOWN: now also U3B.I1
- net !OUT-: now also U3B.I0
- net !UP_DOWN_CLK: now also U19B.I1
- net LCD-13: now also U2B.I0
- net LCD-3: now also U2B.I1; no longer U2B.O
- net N$14: now also U17B.I2, U18D.O; no longer U10A.CO, U6A.D, U6A.S
Other:
- note added: "Clock/ Negative Voltage Generator"
- note added: "Positive Voltage Regulator"
- note added: "Up/Down Counter"
- moved on the sheet: U17B, U18B, U18D, U19D, U2A, U2B, U2D

Commit message: Change reference designators and capacitor values to match 'Official' schematic
Parts:
- removed C22, C23, C24, C25, C27, C28: (no value), rcl:C-EUC0805
- removed D10, D11: 1n4148, diode:DIODE-MINIMELF
- removed R32: 1K, rcl:R-EU_M0805
- removed RX: OPEN, rcl:R-EU_0207/10
- removed X1: 32.768KHz, crystal:CRYSTALTC26H
- added E1, E2, E6: 10uF 63V, rcl:CPOL-EUE2.5-5
- added E3, E4, E5: 47uf 25V, rcl:CPOL-EUE2.5-5
- added M1: IRF740, transistor-power:IRF740
- added R51: 2K, rcl:R-EU_M0805
- added R52: 1K, rcl:R-EU_M0805
- added Z1: 12V, diode:ZENER-DIODESOD80C
- added Z2: 6.2V, diode:ZENER-DIODESOD80C
- C1: value (none) -> 100nF; device rcl:C-EU050-024X044 -> rcl:C-EUC1206
- C10, C12, C13, C14, C16: value (none) -> 100nF
- C11: value (none) -> 220pF; device rcl:C-EUC1206 -> rcl:C-EUC0805
- C15, C8, C9: value (none) -> 10nF; device rcl:C-EUC1206 -> rcl:C-EUC0805
- C17: value (none) -> 10pF; device rcl:C-EU050-045X075 -> rcl:C-EUC0805
- C18: value (none) -> 39pF; device rcl:C-EU050-045X075 -> rcl:C-EUC0805
- C19: value (none) -> 10nF
- C2: value 47uf 25V -> 100nF; device rcl:CPOL-EUE2.5-5 -> rcl:C-EUC1206
- C20: device rcl:C-EUC0805 -> rcl:C-EU050-024X044
- C3, C4: value 47uf 25V -> 1uF; device rcl:CPOL-EUE2.5-5 -> rcl:C-EU050-045X075
- C5, C6: value 10uF 63V -> 100nF; device rcl:CPOL-EUE2.5-5 -> rcl:C-EUC1206
- C7: value 10uF 63V -> 10nF; device rcl:CPOL-EUE2.5-5 -> rcl:C-EUC0805
- D1: value V674 -> 1N4448; device diode:DIODE-SOD80C -> diode:DIODE-MINIMELF
- D2, D4, D7: value 1N4148 -> 1N4448
- D3, D5: value ZENER? -> 1N4448
- D6, D8: value 1n4148 -> 1N4448
- D9: value 1n4148 -> 1N4004; device diode:DIODE-MINIMELF -> diode:DIODE-SOD80C
- F1: value FUSEBLANK_5X20MM -> 32mA
- Q1: value IRF740 -> 32.768KHz; device transistor-power:IRF740 -> crystal:CRYSTALTC26H
- R1: value 20K -> 620
- R10: value 1M -> 3K
- R12, R14: value 1M -> 330K
- R13: value 3K -> 330K
- R16: value 100K -> 1M
- R18, R19: value 300 -> 47
- R2: value 20K -> 300
- R20: value 2K -> 1K
- R21: value 130K -> 10M; device rcl:R-EU_0207/10 -> rcl:R-EU_M0805
- R22: value 130K -> 20K; device rcl:R-EU_0207/10 -> rcl:R-EU_M0805
- R23: value 4.70K -> 100K; device rcl:R-EU_0207/10 -> rcl:R-EU_M0805
- R24: value 8.20K -> 20K; device rcl:R-EU_0207/10 -> rcl:R-EU_M0805
- R25: value 620 -> 100K
- R26: value 47 -> 330K
- R27: value 47 -> 2K
- R28: value 10M -> 2K
- R29: value 330K -> 1M
- R3: value 2K -> 300
- R30: value 1K -> 1M
- R31: value 10K -> OPEN; device rcl:R-EU_M0805 -> rcl:R-EU_0207/10
- R4: value 2K -> 10K
- R5: value 2K -> 130K; device rcl:R-EU_M0805 -> rcl:R-EU_0207/10
- R6: value 100K -> 130K; device rcl:R-EU_M0805 -> rcl:R-EU_0207/10
- R7: value 330K -> 2K
- R8: value 330K -> 4.70K; device rcl:R-EU_M0805 -> rcl:R-EU_0207/10
- R9: value 330K -> 8.20K; device rcl:R-EU_M0805 -> rcl:R-EU_0207/10
- renumbered U1 to IC18, U10 to IC12, U11 to IC3, U12 to IC7, U13 to IC15, U14 to IC17, U15 to IC1, U16 to IC6, U17 to IC16, U18 to IC11, U19 to IC9, U2 to IC19, U3 to IC14, U4 to IC8, U5 to IC10, U6 to IC13, U7 to IC2, U8 to IC4, U9 to IC5
Connections:
- net !NAR: now also R22.1; no longer R1.1
- net !NAR_R: now also C15.1, R22.2, R23.1; no longer C19.1, R1.2, R6.1
- net !RESET: now also R24.1; no longer R2.1
- net +5V: now also C12.1, C19.1, E3.+, R11.2, R19.2, Z1.A, Z2.C; no longer C2.+, C24.1, C8.1, D3.A, D4.C, R12.2, R26.2
- net -1V25: now also C8.1, C9.2, R13.1, R14.2; no longer C20.2, C21.1, R7.2, R8.1
- net -2V5: now also C9.1, R14.1; no longer C20.1, R7.1
- net -2V5_BUF: now also R10.2; no longer R13.2
- net -2V5_BUF_R: now also R10.1; no longer R13.1
- net -4V: now also D6.A, E4.-; no longer C4.-, D11.A
- net -5V: now also C13.1, R18.1; no longer C16.1, R27.1
- net 0V0: now also C8.2, R12.1, R13.2; no longer C21.2, R8.2, R9.1
- net 13V5: now also D8.A, E2.+, M1.S; no longer C5.+, D2.A, Q1.S
- net 1V25: now also C7.2, R11.1, R12.2; no longer C22.2, R12.1, R9.2
- net 2_048KHZ: now also E5.+; no longer C3.+
- net 32_768KHZ: now also R21.1, R26.1; no longer R28.1, R29.1
- net AH_NEGATIVE: now also R51.1; no longer R3.1
- net AH_NEGATIVE_R: now also R23.2, R51.2; no longer R3.2, R6.2
- net CXA: now also C5.1; no longer C13.1
- net CXB: now also C6.1; no longer C14.1
- net DRAIN: now also D9.C, M1.D; no longer D1.C, Q1.D
- net FUSED_BATT+: now also D9.A, R30.2; no longer D1.A, R14.2
- net GATE: now also C21.1, D8.C, M1.G, R29.2, Z1.C; no longer C23.1, D2.C, D3.C, Q1.G, R15.2
- net GND: now also C10.2, C17.1, C18.1, C20.2, C21.2, C3.2, C4.2, C5.2, C6.2, C7.1, D1.C, D2.A, D3.C, D5.C, D7.A, E2.-, E3.-, E4.+, E6.-, R52.2, Z2.A; no longer C1.2, C17.2, C18.2, C2.-, C22.1, C23.2, C24.2, C27.1, C28.1, C4.+, C5.-, C7.-, C8.2, C9.2, D10.C, D5.A, D6.A, D7.C, D8.A, D9.C, R30.2
- net GND1K: now also R52.1; no longer R30.1
- net IN+: now also C3.1, D1.A, D2.C, R1.2; no longer C17.1, D8.C, D9.A, R25.2
- net IN-: now also C1.1, C2.1, D3.A, D4.C, R3.2, R31.2, R4.1, R5.2, R7.1, R8.2; no longer C10.1, C11.1, D6.C, D7.A, R19.2, R20.1, R21.2, R23.2, R31.1, RX.2
- net LCD-20: now also D7.C, E1.-; no longer C6.-, D5.C
- net LCD-3: now also C20.1; no longer C1.1
- net N$13: now also C11.2; no longer C25.2
- net N$24: now also C11.1; no longer C25.1
- net N$29: now also R29.1, R30.1; no longer R14.1, R15.1
- net N$32: now also R20.2; no longer R32.2
- net N$38: now also D5.A, D6.C, E5.-; no longer C3.-, D10.A, D11.C
- net N$39: now also C17.2, Q1.1, R26.2; no longer C27.2, R29.2, X1.1
- net N$40: now also C18.2, Q1.2, R21.2; no longer C28.2, R28.2, X1.2
- net N$42: now also R5.1, R6.2; no longer R21.1, R22.2
- net N$45: now also R8.1, R9.2; no longer R23.1, R24.2
- net N$48: now also R25.1; no longer R16.1
- net N$53: now also R15.2; no longer R11.2
- net N$54: now also E1.+, R20.1; no longer C6.+, R32.1
- net N$55: now also R16.1; no longer R10.1
- net N$56: now also R15.1; no longer R11.1
- net N$57: now also R16.2; no longer R10.2
- net OUT: now also C1.2, C2.2; no longer C10.2, C11.2
- net OUT+: now also R28.1; no longer R4.1
- net OUT+_R: now also R28.2; no longer R4.2
- net OUT-: now also R27.1; no longer R5.1
- net OUT-_R: now also R27.2; no longer R5.2
- net RESET_R: now also C16.1, E6.+, R24.2, R25.2; no longer C7.+, C9.1, R16.2, R2.2
- net SHUNT+: now also R2.1; no longer R18.1
- net SHUNT+FILTER: now also C4.1, R2.2, R3.1; no longer C18.1, R18.2, R19.1
- net SHUNT-: now also R1.1; no longer R25.1
- net VDD+: now also C10.1, R19.1; no longer C15.1, R26.1
- net VDD-: now also C14.1, R18.2; no longer C12.1, R27.2
- net X0: now also R31.1, R7.2, R9.1; no longer R20.2, R24.1, RX.1
- net Y0: now also R4.2, R6.1; no longer R22.1, R31.2
Other:
- moved on the sheet: C1, C10, C11, C12, C13, C14, C15, C16, C17, C18, C19, C20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

Commit message: update lcd interface portion
Parts:
- C20, C21: value (none) -> 10nF
Connections:
- net AH_NEGATIVE_R renamed MINUS_SIGN_ON
- net LCD-10 renamed LCD_ONE_MSD
- net LCD-11 renamed LCD_COLON
- net LCD-17 renamed !LCD_RESET
- net LCD-19 renamed LCD_45_HZ
- net LCD-20 renamed V_F_OUT
- net LCD-7 renamed LCD_DECIMAL_POINT
- net LCD-8 renamed LCD_MINUS_SIGN
- net LCD-9 renamed OVER_FLOW_UP
- net N$14 renamed IC3-11
- net U12-14 renamed IC7-14
- net U13-12 renamed IC15-12
- net U13-13 renamed OVER_FLOW
- net U13-3 renamed IC15-3
- net U17-2 renamed IC16-2
- net U3-6 renamed IC14-6
- net U4-3 renamed IC8-3
- net U5-7 renamed IC10-7
- net U6-5 renamed IC13-5
- net U9-4 renamed IC5-4
- removed net N$22: IC9A.I1, IC9D.O
- removed net U14-1: IC17A.I0, IC9B.O, IC9C.I1
- new net COLON_ON: IC17A.I0
- new net IC17-1: IC9B.O, IC9C.I1
- net +5V: now also IC3P.VCC
- net -5V: now also IC3P.VEE
- net AH_NEGATIVE_LCD: now also IC9A.I1, IC9D.O
- net GND: now also IC3P.GND
Other:
- note added: "Blanks 4 LSD"
- note added: "Count Zero"
- note added: "Overflow?"
- note added: "To LCD Module"
- note removed: "LCD"
- moved on the sheet: C11, IC11B, IC11D, IC14A, IC15A, IC15B, IC16B, IC16C, IC17A, IC17B, IC17C, IC17D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
